File: eagle_NAHS-RHTBrick/v1.0_r1.brd (EAGLE design)
At the start: 45.5 x 70.3 mm, 47 parts, among them IC1 ESP12S, IC2 ATTINY212-SSNR, IC3 TP4056, IC4 DW01A, IC5 HDC1080, J1 10118194-0001LF, J2 BRICK-INTERF-V3_B-SIDE, Q1 8205A, T1 PINHD_1X03_R_1, T2 PINHD_1X03_R_1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

Commit message: saving
Connections:
- net GND: no longer IC5.7, IC5.7.1, IC5.7.2, IC5.7.3, IC5.7.4
Routing:
- net 1WIRE: track 22.5 -> 48.0 mm, vias 0 -> 1
- net GND: track 176.7 -> 177.8 mm
Changed lines of the file:
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@@
 <setting verticaltext="up"/>
 </settings>
-<grid distance="25" unitdist="mil" unit="mil" style="lines" multiple="1" display="yes" altdistance="5" altunitdist="mil" altunit="mil"/>
+<grid distance="25" unitdist="mil" unit="mm" style="lines" multiple="1" display="yes" altdistance="5" altunitdist="mil" altunit="mil"/>
 <layers>
 <layer number="1" name="Top" color="4" fill="1" visible="yes" active="yes"/>
@@
 </class>
 </classes>
-<designrules name="JLCPCB">
+<designrules name="JLCPCB *">
 <description language="de">&lt;b&gt;EAGLE Design Rules&lt;/b&gt;
 &lt;p&gt;
@@
 <param name="rvMicroViaOuter" value="0.25"/>
 <param name="rvMicroViaInner" value="0.25"/>
-<param name="rlMinPadTop" value="10mil"/>
+<param name="rlMinPadTop" value="0.13mm"/>
 <param name="rlMaxPadTop" value="20mil"/>
 <param name="rlMinPadInner" value="10mil"/>
 <param name="rlMaxPadInner" value="20mil"/>
-<param name="rlMinPadBottom" value="10mil"/>
+<param name="rlMinPadBottom" value="0.13mm"/>
 <param name="rlMaxPadBottom" value="20mil"/>
-<param name="rlMinViaOuter" value="8mil"/>
+<param name="rlMinViaOuter" value="0.13mm"/>
 <param name="rlMaxViaOuter" value="20mil"/>
 <param name="rlMinViaInner" value="8mil"/>
@@
 <wire x1="30.861" y1="47.26575" x2="30.861" y2="50.673" width="0.4064" layer="1"/>
 <wire x1="30.243325" y1="46.648075" x2="30.861" y2="47.26575" width="0.4064" layer="1"/>
-<wire x1="30.243325" y1="45.067675" x2="30.243325" y2="46.648075" width="0.4064" layer="1"/>
+<wire x1="30.243325" y1="45.067675" x2="30.243325" y2="45.085" width="0.4064" layer="1"/>
+<wire x1="30.243325" y1="45.085" x2="30.243325" y2="46.648075" width="0.4064" layer="1"/>
 <wire x1="31.496" y1="43.815" x2="30.243325" y2="45.067675" width="0.4064" layer="1"/>
 <wire x1="40.23173125" y1="48.6184" x2="43.88613125" y2="44.964" width="0.254" layer="1"/>
@@
 <wire x1="43.88613125" y1="44.964" x2="43.88613125" y2="29.877" width="0.254" layer="1"/>
 <contactref element="IC5" pad="2"/>
-<contactref element="IC5" pad="7.1"/>
-<contactref element="IC5" pad="7"/>
-<contactref element="IC5" pad="7.3"/>
-<contactref element="IC5" pad="7.4"/>
-<contactref element="IC5" pad="7.2"/>
 <contactref element="T1" pad="3"/>
 <contactref element="T2" pad="3"/>
@@
 <wire x1="38.1" y1="40.005" x2="38.1" y2="33.655" width="0.4064" layer="16"/>
 <wire x1="38.1" y1="27.305" x2="38.1" y2="33.655" width="0.4064" layer="16"/>
-<wire x1="38.1" y1="27.305" x2="32.618" y2="21.823" width="0.4064" layer="16"/>
-<wire x1="32.618" y1="21.823" x2="29.824" y2="21.823" width="0.4064" layer="16"/>
 <contactref element="RHT-ALT" pad="1"/>
 <wire x1="19.7838" y1="30.78395" x2="19.7838" y2="32.4838" width="0.4064" layer="16"/>
@@
 <wire x1="22.86" y1="32.385" x2="22.86" y2="35.56" width="0.254" layer="1"/>
 <wire x1="24.395" y1="30.85" x2="22.86" y2="32.385" width="0.254" layer="1"/>
-<wire x1="25.27" y1="30.85" x2="26.17" y2="30.85" width="0.254" layer="1"/>
 <contactref element="C6" pad="2"/>
 <wire x1="25.72" y1="27.94" x2="24.395" y2="29.265" width="0.254" layer="1"/>
 <wire x1="24.395" y1="29.265" x2="24.395" y2="30.85" width="0.254" layer="1"/>
-<wire x1="27.17" y1="30.85" x2="26.67" y2="30.85" width="0" layer="19" extent="1-1"/>
-<wire x1="26.17" y1="30.85" x2="26.67" y2="30.85" width="0" layer="19" extent="1-1"/>
-<wire x1="26.67" y1="31.8" x2="26.67" y2="30.85" width="0" layer="19" extent="1-1"/>
-<wire x1="26.67" y1="29.9" x2="26.67" y2="30.85" width="0" layer="19" extent="1-1"/>
+<wire x1="30.243325" y1="45.067675" x2="30.243325" y2="42.943325" width="0.4064" layer="1"/>
+<wire x1="30.243325" y1="42.943325" x2="22.86" y2="35.56" width="0.4064" layer="1"/>
+<polygon width="0.1524" layer="1" pour="cutout">
+<vertex x="23.495" y="24.765"/>
+<vertex x="40.005" y="24.765"/>
+<vertex x="40.005" y="42.545"/>
+<vertex x="31.115" y="42.545"/>
+<vertex x="23.495" y="34.925"/>
+</polygon>
+<polygon width="0.1524" layer="16" pour="cutout" rank="2">
+<vertex x="23.495" y="34.925"/>
+<vertex x="23.495" y="24.765"/>
+<vertex x="40.005" y="24.765"/>
+<vertex x="40.005" y="42.545"/>
+<vertex x="31.115" y="42.545"/>
+</polygon>
 </signal>
 <signal name="SEL+">
@@
 <contactref element="IC1" pad="GPIO14"/>
 <wire x1="21.27" y1="17.78" x2="21.59" y2="17.78" width="0.254" layer="1"/>
-<wire x1="31.063" y1="15.823" x2="42.19" y2="15.823" width="0.254" layer="1"/>
+<wire x1="31.063" y1="15.823" x2="32.385" y2="15.823" width="0.254" layer="1"/>
+<wire x1="32.385" y1="15.823" x2="42.19" y2="15.823" width="0.254" layer="1"/>
 <wire x1="21.59" y1="17.78" x2="24.511" y2="14.859" width="0.254" layer="1"/>
 <wire x1="24.511" y1="14.859" x2="30.099" y2="14.859" width="0.254" layer="1"/>
 <wire x1="30.099" y1="14.859" x2="31.063" y2="15.823" width="0.254" layer="1"/>
 <contactref element="T3" pad="2"/>
-<wire x1="35.56" y1="33.655" x2="35.56" y2="40.005" width="0" layer="19" extent="1-1"/>
-<wire x1="35.56" y1="27.305" x2="35.56" y2="33.655" width="0" layer="19" extent="1-1"/>
-<wire x1="42.19" y1="15.823" x2="35.56" y2="27.305" width="0" layer="19" extent="1-1"/>
+<wire x1="35.56" y1="27.305" x2="35.56" y2="18.998" width="0.254" layer="16"/>
+<wire x1="35.56" y1="18.998" x2="32.385" y2="15.823" width="0.254" layer="16"/>
+<via x="32.385" y="15.823" extent="1-16" drill="0.35"/>
+<wire x1="35.56" y1="27.305" x2="35.56" y2="33.655" width="0.254" layer="16"/>
+<wire x1="35.56" y1="33.655" x2="35.56" y2="40.005" width="0.254" layer="16"/>
 </signal>
 <signal name="N$5">

Commit message: v1.0 R1 Board done
Parts:
- removed R16: 590k, rcl:R0805
- removed R17: 2.7M, rcl:R0805
- added R4, R5: 1k, rcl:R0805
- C2: value 1µF -> 100nF
- C4: value 10µF -> 1µF
- C6: value 100nF -> 10µF
- R10, R11: value 3.9k -> 10k
- R14: value 10k -> 590k
- R15: value 10k -> 2.7M
- R3: value 3.9k -> 1k
- R6: value 1k -> 1.74k
- R7, R8: value 1k -> 3.9k
- R9: value 1.74k -> 3.9k
- moved R9 52.3 mm to (20.3, 12.7)
- moved R13 44.4 mm to (29.5, 63.8), turned to 90 degrees
- moved R7 34.8 mm to (20.3, 17.8), turned to 0 degrees
- moved R14 31.1 mm to (34.2, 50.7), turned to 180 degrees
- moved C2 28.0 mm to (26.7, 27.9), turned to 180 degrees
- moved R3 27.3 mm to (27.7, 44.1), turned to 270 degrees
- moved R6 20.8 mm to (25.4, 64.8), turned to 0 degrees
- moved C6 17.7 mm to (20.3, 44.5), turned to 90 degrees
- moved R15 16.0 mm to (38.7, 50.7), turned to 180 degrees
- moved R12 12.7 mm to (20.3, 22.9)
- moved C4 10.7 mm to (30.9, 53.7), turned to 90 degrees
- moved R11 7.62 mm to (20.3, 20.3)
- moved R8 7.62 mm to (20.3, 15.2), turned to 0 degrees
- moved C5 7.62 mm to (20.3, 52.1), turned to 270 degrees
- moved C3 6.86 mm to (37.7, 53.7)
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Connections:
- net +3V3: now also C4.1, R7.1, R8.1, R9.1; no longer C3.1, R12.1, R13.1, R3.1
- net 1WIRE: now also R7.2; no longer R3.2
- net A0: now also R14.1, R15.2; no longer R16.1, R17.2
- net BAT+: now also C6.1; no longer C5.1
- net BAT-: now also R3.1; no longer R6.1
- net BOOT1: now also R11.2; no longer R13.2
- net BOOT2: now also R12.2; no longer R14.2
- net CD: now also R13.2; no longer R15.2
- net CHRG: now also R4.2; no longer R7.2
- net EN: now also R10.2; no longer R12.2
- net GND: now also C4.2, R12.1, R14.2; no longer C6.2, R14.1, R16.2
- net IN-: now also C6.2, R6.1; no longer C4.2, R9.1
- net N$1: now also C5.1, R13.1; no longer C4.1, R15.1
- net N$2: now also R6.2; no longer R9.2
- net N$3: now also R3.2; no longer R6.2
- net N$5: now also C2.1; no longer C6.1
- net N$7: now also R4.1; no longer R7.1
- net RST: now also R5.2; no longer R8.2
- net SCL: now also R9.2; no longer R11.2
- net SDA: now also R8.2; no longer R10.2
- net SEL+: now also C3.1, R15.1; no longer C2.1, R17.1
- net WAKE: now also R5.1; no longer R8.1
Routing:
- net GND: vias 1 -> 2
- added copper zone on layer 1, net N$1
