File: eagle_NAHS-RHTBrick/v1.0_r2.brd (EAGLE design)
At the start: 45.5 x 70.3 mm, 48 parts, among them IC1 ESP12S, IC2 ATTINY212-SSNR, IC3 TP4056, IC4 DW01A, IC5 HDC1080, J1 10118194-0001LF, J2 BRICK-INTERF-V3_B-SIDE, Q1 8205A, T1 PINHD_1X03_R_1, T2 PINHD_1X03_R_1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

Commit message: v1.0 R2 Board done
Parts:
- removed R: KMR_231_G_LFS, no_reichelt:KMR_231_G_LFS
- added S2: KMR_231_G_LFS, no_reichelt:KMR_231_G_LFS
- moved T1 0.63 mm to (36.2, 27.3)
- moved T2 0.63 mm to (36.2, 33.7)
- moved T3 0.63 mm to (36.2, 40.0)
Connections:
- net GND: now also S2.3, S2.4; no longer R.3, R.4
- net RST: now also S2.1, S2.2; no longer R.1, R.2
Routing:
- net RST: track 60.5 -> 33.7 mm, vias 2 -> 0
- net GND: track 177.8 -> 171.6 mm
- net +3V3: track 150.2 -> 150.8 mm
Other:
- board text added: "RST"
