File: eagle_NAHS-RHTBrick/v1.0_r2.sch (EAGLE design)
At the start: 44 parts, among them IC1 ESP12S, IC2 ATTINY212-SSNR, IC3 TP4056, IC4 DW01A, IC5 HDC1080, J1 10118194-0001LF, J2 BRICK-INTERF-V3_B-SIDE, Q1 8205A, T1 PINHD_1X03_R_1, T2 PINHD_1X03_R_1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

Commit message: v1.0 R2 Board done
Parts:
- renumbered R to S2
Changed lines of the file:
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@@
 <part name="R4" library="rcl" library_urn="urn:adsk.eagle:library:334" deviceset="R-EU_" device="R0805" package3d_urn="urn:adsk.eagle:package:23553/2" value="1k"/>
 <part name="JP2" library="no_pinhd" deviceset="PINHD_1X03" device="_R_1"/>
-<part name="R" library="no_reichelt" deviceset="KMR_231_G_LFS" device=""/>
+<part name="S2" library="no_reichelt" deviceset="KMR_231_G_LFS" device=""/>
 <part name="GND5" library="supply1" library_urn="urn:adsk.eagle:library:371" deviceset="GND" device=""/>
 <part name="+3V4" library="supply1" library_urn="urn:adsk.eagle:library:371" deviceset="+3V3" device=""/>
@@
 <attribute name="NAME" x="95.885" y="76.2" size="1.27" layer="95" rot="R180" align="center-left"/>
 </instance>
-<instance part="R" gate="G$1" x="99.06" y="66.04" smashed="yes" rot="R270" grouprefs="MAINIC">
+<instance part="S2" gate="G$1" x="99.06" y="66.04" smashed="yes" rot="R270" grouprefs="MAINIC">
 <attribute name="VALUE" x="93.98" y="71.12" size="1.27" layer="96"/>
 <attribute name="NAME" x="93.98" y="63.5" size="1.27" layer="95"/>
@@
 <wire x1="86.36" y1="66.04" x2="88.9" y2="66.04" width="0.1524" layer="91" grouprefs="MAINIC"/>
 <junction x="88.9" y="66.04" grouprefs="MAINIC"/>
-<pinref part="R" gate="G$1" pin="2"/>
+<pinref part="S2" gate="G$1" pin="2"/>
 <wire x1="93.98" y1="66.04" x2="88.9" y2="66.04" width="0.1524" layer="91" grouprefs="MAINIC"/>
 </segment>
@@
 </segment>
 <segment>
-<pinref part="R" gate="G$1" pin="1"/>
+<pinref part="S2" gate="G$1" pin="1"/>
 <wire x1="104.14" y1="66.04" x2="106.68" y2="66.04" width="0.1524" layer="91" grouprefs="MAINIC"/>
 <label x="106.68" y="66.04" size="1.778" layer="95" xref="yes" grouprefs="MAINIC"/>
