File: kicad/nahs-RHTBrick_v1.0_panel/nahs-RHTBrick_v1.0_panel.kicad_sch (KiCad schematic)
At the start: 68 parts, among them IC1 ESP12S, IC2 ATTINY212, J2 USB_B_Mini, Q1 8205A, Q3 CJ2302, Q4 MMBT2907A, SW1 KMR_231_G_LFS, SW2 SSSS820101, U1 ZD8028IB5TR, U2 HDC1080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

Commit message: v1.0 Board done; v1.0 Breakout Board done
Parts:
- BT, J2: Handsolder true -> (none)
- C1: DNP (none) -> true
- L1, Q1, U3, U4: Storage MAG4 -> MAG5
Changed lines of the file:
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@@
       (effects (font (size 1.27 1.27)) hide)
     )
-    (property "Storage" "MAG4" (id 4) (at 266.7 38.1 0)
+    (property "Storage" "MAG5" (id 4) (at 266.7 38.1 0)
       (effects (font (size 1.27 1.27)) hide)
     )
@@
       (effects (font (size 1.27 1.27)) hide)
     )
-    (property "Handsolder" "true" (id 6) (at 85.09 157.48 0)
-      (effects (font (size 1.27 1.27)) hide)
-    )
     (pin "1")
     (pin "2")
@@
       (effects (font (size 1.27 1.27)) hide)
     )
-    (property "Handsolder" "true" (id 8) (at 134.62 85.09 0)
-      (effects (font (size 1.27 1.27)) hide)
-    )
     (pin "M")
     (pin "P")
@@
       (effects (font (size 1.27 1.27)) hide)
     )
-    (property "Storage" "MAG4" (id 4) (at 149.86 128.27 0)
+    (property "Storage" "MAG5" (id 4) (at 149.86 128.27 0)
       (effects (font (size 1.27 1.27)) hide)
     )
@@
       (effects (font (size 1.27 1.27)) hide)
     )
-    (property "Storage" "MAG4" (id 4) (at 247.65 38.1 0)
+    (property "Storage" "MAG5" (id 4) (at 247.65 38.1 0)
       (effects (font (size 1.27 1.27)) hide)
     )
@@
       (effects (font (size 1.27 1.27)) hide)
     )
-    (property "Storage" "MAG4" (id 7) (at 184.15 36.83 0)
+    (property "Storage" "MAG5" (id 7) (at 184.15 36.83 0)
       (effects (font (size 1.27 1.27)) hide)
     )
@@
       (effects (font (size 1.27 1.27)) hide)
     )
-    (property "DNP" "" (id 8) (at 63.5 119.38 0)
-      (effects (font (size 1.27 1.27)) hide)
-    )
+    (property "DNP" "true" (id 8) (at 63.5 119.38 0)
+      (effects (font (size 1.27 1.27)) hide)
+    )
