File: kicad/nahs-RHTBrick_v1.0/nahs-RHTBrick_v1.0.kicad_sch (KiCad schematic)
At the start: 68 parts, among them IC1 ESP12S, IC2 ATTINY212, J2 USB_B_Mini, Q1 8205A, Q3 CJ2302, Q4 MMBT2907A, SW1 KMR_231_G_LFS, SW2 SSSS820101, U1 ZD8028IB5TR, U2 HDC1080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

Commit message: updated footprints for stencil
Parts:
- J2: footprint Connector_USB:USB_Micro-B_Amphenol_10118194_Horizontal -> no_common:USB_Micro-B_Amphenol_10118194_Horizontal
Changed lines of the file:
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@@
     (property "Reference" "J2" (id 0) (at 85.09 144.78 0))
     (property "Value" "USB_B_Mini" (id 1) (at 85.09 147.32 0))
-    (property "Footprint" "Connector_USB:USB_Micro-B_Amphenol_10118194_Horizontal" (id 2) (at 88.9 158.75 0)
+    (property "Footprint" "no_common:USB_Micro-B_Amphenol_10118194_Horizontal" (id 2) (at 88.9 158.75 0)
       (effects (font (size 1.27 1.27)) hide)
     )
@@
     )
     (path "/37c4d311-ec8e-417b-aba7-859c05b65d7b"
-      (reference "J2") (unit 1) (value "USB_B_Mini") (footprint "Connector_USB:USB_Micro-B_Amphenol_10118194_Horizontal")
+      (reference "J2") (unit 1) (value "USB_B_Mini") (footprint "no_common:USB_Micro-B_Amphenol_10118194_Horizontal")
     )
     (path "/6eee5d3c-5ddb-4e02-ba96-6197435dd0af"
